Commit message: updating to add maciv2

File: robot_description/maciv2.urdf.xacro (robot description, xacro)
@@ -2,4 +2,5 @@
 <robot xmlns:xacro="http://www.ros.org/wiki/xacro" name="maciv2">
     <!-- Robot stuff goes here -->
+    <xacro:include filename="$(find krytn)/robot_description/magni/inertial.xacro" />
     <xacro:include filename="$(find ur_description)/urdf/ur_macro.xacro" />
     <xacro:arg name="ur_type" default="ur5e"/>
@@ -8,3 +9,64 @@
     </xacro:ur_robot>
     <link name="world" />
+    <joint name="gripper_joint" type="fixed">
+        <parent link="ur5_tool0" />
+        <child link="Link" />
+        <origin xyz="0 0 0" rpy="0 ${pi/2} 0" />
+    </joint>
+    <link name="Link">
+        <visual>
+            <!--gripper_base-->
+            <geometry>
+                <mesh filename="file://$(find maciv2)/robot_description/meshes/Unnamed_gripper_base.dae"/>
+            </geometry>
+        </visual>
+        <collision>
+            <!--gripper_base-->
+            <geometry>
+                <mesh filename="file://$(find maciv2)/robot_description/meshes/Unnamed_gripper_base.dae"/>
+            </geometry>
+        </collision>
+    </link>
+    <link name="Link001">
+        <visual>
+            <!--finger-->
+            <origin rpy="0.0 -0.0 0.0" xyz="0.0 0.0 0.0"/>
+            <geometry>
+                <mesh filename="file://$(find maciv2)/robot_description/meshes/Unnamed_finger.dae"/>
+            </geometry>
+        </visual>
+        <collision>
+            <!--finger-->
+            <origin rpy="0.0 -0.0 0.0" xyz="0.0 0.0 0.0"/>
+            <geometry>
+                <mesh filename="file://$(find maciv2)/robot_description/meshes/Unnamed_finger.dae"/>
+            </geometry>
+        </collision>
+        <xacro:box_inertial x="0.03" y="0.03" z="0.1" mass="1" />
+    </link>
+    <joint name="finger_joint" type="prismatic">
+        <parent link="Link"/>
+        <child link="Link001"/>
+        <origin rpy="0.0 -0.0 0.0" xyz="-0.13 0 -0.1"/>
+        <axis xyz="0 0 1"/>
+        <limit effort="1000.0" lower="-0.08" upper="0.0" velocity="2.2"/>
+    </joint>
+    <!-- Configure Control of Joints -->
+    <ros2_control name="maciv2" type="system">
+        <hardware>
+            <plugin>ign_ros2_control/IgnitionSystem</plugin>
+        </hardware>
+        <joint name="finger_joint">
+            <command_interface name="position"/>
+            <state_interface name="position">
+                <param name="initial_value">0.0</param>
+            </state_interface>
+            <state_interface name="velocity"/>
+        </joint>
+    </ros2_control>
+    <gazebo>
+        <plugin filename="ign_ros2_control-system" name="ign_ros2_control::IgnitionROS2ControlPlugin">
+            <parameters>$(find maci)/config/ros2_control.yaml</parameters>
+        </plugin>
+    </gazebo>
 </robot>

Commit message: Configuration with setup wizard and auto program to controll gripper

File: robot_description/maciv2.urdf.xacro (robot description, xacro)
@@ -48,7 +48,7 @@
         <parent link="Link"/>
         <child link="Link001"/>
-        <origin rpy="0.0 -0.0 0.0" xyz="-0.13 0 -0.1"/>
+        <origin rpy="0.0 -0.0 0.0" xyz="-0.115 0 -0.05"/>
         <axis xyz="0 0 1"/>
-        <limit effort="1000.0" lower="-0.08" upper="0.0" velocity="2.2"/>
+        <limit effort="1000.0" lower="0.0" upper="0.064" velocity="2.2"/>
     </joint>
     <!-- Configure Control of Joints -->
@@ -67,5 +67,5 @@
     <gazebo>
         <plugin filename="ign_ros2_control-system" name="ign_ros2_control::IgnitionROS2ControlPlugin">
-            <parameters>$(find maci)/config/ros2_control.yaml</parameters>
+            <parameters>$(find maciv2)/config/ros2_controllers.yaml</parameters>
         </plugin>
     </gazebo>

Commit message: Maciv2 Cokeworls and auto program to pickup and drop of can

File: robot_description/maciv2.urdf.xacro (robot description, xacro)
@@ -2,4 +2,9 @@
 <robot xmlns:xacro="http://www.ros.org/wiki/xacro" name="maciv2">
     <!-- Robot stuff goes here -->
+   <xacro:include filename="$(find realsense2_description)/urdf/_d435i.urdf.xacro" />
+  <!-- Including realsense description from external package -->
+    <xacro:sensor_d435i parent="ur5_base_link" name="sensor_d435i" use_nominal_extrinsics="True">
+        <origin xyz="-1 -1 0.5" rpy="0 0 ${pi/4}"/>
+    </xacro:sensor_d435i>
     <xacro:include filename="$(find krytn)/robot_description/magni/inertial.xacro" />
     <xacro:include filename="$(find ur_description)/urdf/ur_macro.xacro" />
@@ -69,4 +74,38 @@
             <parameters>$(find maciv2)/config/ros2_controllers.yaml</parameters>
         </plugin>
+        <plugin filename="ignition-gazebo-sensors-system" name="ignition::gazebo::systems::Sensors">
+            <render_engine>ogre2</render_engine>
+        </plugin>
+    </gazebo>
+ <!-- Add sensor tags to Realsense links -->
+    <gazebo reference="sensor_d435i_link">
+        <sensor name="realsense_d435" type="rgbd_camera">
+            <topic>realsense</topic>
+            <ignition_frame_id>sensor_d435i_link</ignition_frame_id>
+            <update_rate>5</update_rate>
+            <camera name="camera">
+                <horizontal_fov>1.5</horizontal_fov>
+                <image>
+                    <width>320</width>
+                    <height>240</height>
+                    <format>R8G8B8</format>
+                </image>
+                <clip>
+                    <near>0.01</near>
+                    <far>10</far>
+                </clip>
+                <depth_camera>
+                    <clip>
+                        <near>0.1</near>
+                        <far>10</far>
+                    </clip>
+                </depth_camera>
+                <noise>
+                    <type>gaussian</type>
+                    <mean>0</mean>
+                    <stddev>0.007</stddev>
+                </noise>
+            </camera>
+        </sensor>
     </gazebo>
 </robot>
